File: simple_rx.sch (KiCad schematic (older format))
At the start: 68 parts, among them P1 CONN_01X08, P2 CONN_01X08, P3 CONN_01X03, P4 CONN_01X03, U1 TL072, U2 LM7805CT, U3 LM7905CT, U4 TL072

Commit message: line receiver PCB looks complete
Parts:
- added FID1, FID2, FID3, FID4: FIDUCIAL, smd:FID0.5, symbol FIDUCIAL
Changed lines of the file:
@@
 	7500 3800 7500 3900
 Connection ~ 7500 3800
+$Comp
+L FIDUCIAL FID1
+U 1 1 59ECEE78
+P 6950 5150
+F 0 "FID1" H 6950 5150 60  0000 C CNN
+F 1 "FIDUCIAL" H 6950 5350 60  0000 C CNN
+F 2 "smd:FID0.5" H 6950 5150 60  0001 C CNN
+F 3 "" H 6950 5150 60  0000 C CNN
+	1    6950 5150
+	1    0    0    -1
+$EndComp
+$Comp
+L FIDUCIAL FID2
+U 1 1 59ECFDCC
+P 7350 5150
+F 0 "FID2" H 7350 5150 60  0000 C CNN
+F 1 "FIDUCIAL" H 7350 5350 60  0000 C CNN
+F 2 "smd:FID0.5" H 7350 5150 60  0001 C CNN
+F 3 "" H 7350 5150 60  0000 C CNN
+	1    7350 5150
+	1    0    0    -1
+$EndComp
+$Comp
+L FIDUCIAL FID3
+U 1 1 59ECFED8
+P 6950 5550
+F 0 "FID3" H 6950 5550 60  0000 C CNN
+F 1 "FIDUCIAL" H 6950 5750 60  0000 C CNN
+F 2 "smd:FID0.5" H 6950 5550 60  0001 C CNN
+F 3 "" H 6950 5550 60  0000 C CNN
+	1    6950 5550
+	1    0    0    -1
+$EndComp
+$Comp
+L FIDUCIAL FID4
+U 1 1 59ED00C0
+P 7350 5550
+F 0 "FID4" H 7350 5550 60  0000 C CNN
+F 1 "FIDUCIAL" H 7350 5750 60  0000 C CNN
+F 2 "smd:FID0.5" H 7350 5550 60  0001 C CNN
+F 3 "" H 7350 5550 60  0000 C CNN
+	1    7350 5550
+	1    0    0    -1
+$EndComp
 $EndSCHEMATC
